Commit message: joint1 lined up

File: urdf/robot_description.urdf (robot description, URDF)
Before this commit: robot visual, 4 links, 3 joints
Joints:
- removed joint BaseToLink2
- removed joint Link2ToLink3
- removed joint Link3ToLink4
- added joint joint0: type revolute, parent base_link, child Link2, origin xyz=0 -0.06 .159 rpy= 0 0 3.14159, axis 0 0 1, limit lower=0 upper=6 effort=1.0 velocity=1.0
- added joint joint1: type revolute, parent Link2, child Link3, origin xyz=0.07 0 0 rpy= 0 0 0, axis 0 1 0, limit lower=0 upper=6 effort=1.0 velocity=1.0
- added joint joint2: type revolute, parent Link3, child Link4, origin xyz=-0.17 -0.025 0 rpy= 0 0 0, axis 0 1 0, limit lower=0 upper=6 effort=1.0 velocity=1.0

Commit message: urdf has right frames but wrong link lengths

File: urdf/robot_description.urdf (robot description, URDF)
Before this commit: robot visual, 4 links, 3 joints
Links:
- added link Link1
- link Link2: geometry 
- link Link3: geometry 
- link Link4: geometry 
- link base_link: geometry 
Joints:
- added joint EE: type fixed, parent Link3, child Link4, origin xyz=.5 0 0 rpy= 0 0 0, axis 0 0 1, limit lower=0 upper=6 effort=1.0 velocity=1.0
- joint joint0: child Link2 -> Link1; origin xyz=0 -0.06 .159 rpy= 0 0 3.14159 -> xyz=0 0 0 rpy= 0 0 0
- joint joint1: axis 0 1 0 -> 0 0 1; child Link3 -> Link2; origin xyz=0.07 0 0 rpy= 0 0 0 -> xyz=0 0 .08 rpy=-1.57 0 0; parent Link2 -> Link1
- joint joint2: axis 0 1 0 -> 0 0 1; child Link4 -> Link3; origin xyz=-0.17 -0.025 0 rpy= 0 0 0 -> xyz=.5 0 0 rpy= 0 0 0; parent Link3 -> Link2

Commit message: correct link lengths???

File: urdf/robot_description.urdf (robot description, URDF)
Before this commit: robot visual, 5 links, 4 joints
Links:
- removed link Link4
- added link EE
Joints:
- joint EE: child Link4 -> EE; origin xyz=.5 0 0 rpy= 0 0 0 -> xyz=.24 0 0 rpy= 0 0 0
- joint joint1: origin xyz=0 0 .08 rpy=-1.57 0 0 -> xyz=0 0 .168 rpy=-1.57 0 0
- joint joint2: origin xyz=.5 0 0 rpy= 0 0 0 -> xyz=.24 0 0 rpy= 0 0 0
