Commit message: add test files

File: urdf/hephaestus.urdf.xacro (robot description, xacro)
@@ -10,5 +10,5 @@
         <parent link="base_link"/>
         <child link="${prefix}_link1"/>
-        <origin xyz="0 ${reflect*(.5)} 0" />
+        <origin xyz="0 ${reflect*(0)} 0" />
         <limit effort="1.0" lower="0" upper="6" velocity="1.0"/>
         <axis xyz = "0 0 1"/>

File: urdf/strokearm.urdf.xacro (robot description, xacro)
@@ -8,4 +8,4 @@
 </link>
 <xacro:hephaestus prefix="master" reflect="1" />
-<xacro:hephaestus prefix="slave" reflect="-1" />
+<!-- <xacro:hephaestus prefix="slave" reflect="-1" /> -->
 </robot>

Commit message: working

File: urdf/hephaestus.urdf.xacro (robot description, xacro)
@@ -10,5 +10,5 @@
         <parent link="base_link"/>
         <child link="${prefix}_link1"/>
-        <origin xyz="0 ${reflect*(0)} 0" />
+        <origin xyz="0 ${reflect*(0)} 0" rpy="0 0.785 0"/>
         <limit effort="1.0" lower="0" upper="6" velocity="1.0"/>
         <axis xyz = "0 0 1"/>

Commit message: fixed things

File: urdf/hephaestus.urdf.xacro (robot description, xacro)
@@ -32,5 +32,5 @@
     </link>
     <joint name="${prefix}_joint2" type="revolute">
-      <origin xyz=".24 0 0" rpy=" 0 0 0"/>
+      <origin xyz=".24 0 0" rpy="0 0 1.57"/>
       <parent link="${prefix}_link2"/>
       <child link="${prefix}_link3"/>

Commit message: both arms working

File: urdf/hephaestus.urdf.xacro (robot description, xacro)
@@ -10,5 +10,5 @@
         <parent link="base_link"/>
         <child link="${prefix}_link1"/>
-        <origin xyz="0 ${reflect*(0)} 0" rpy="0 0.785 0"/>
+        <origin xyz="0 ${reflect} 0" rpy="0 0.785 0"/>
         <limit effort="1.0" lower="0" upper="6" velocity="1.0"/>
         <axis xyz = "0 0 1"/>

File: urdf/strokearm.urdf.xacro (robot description, xacro)
@@ -2,5 +2,5 @@
 <robot xmlns:xacro="http://www.ros.org/wiki/xacro" name="stroke">
 <xacro:include filename="hephaestus.urdf.xacro"/>
-<xacro:arg name="twoArm" default="false"/>
+<xacro:arg name="twoArm" default="true"/>
 <link name="base_link">
 <origin xyz="0 0 0 " rpy=" 0 0 0"/>
@@ -8,8 +8,8 @@
         </visual>
 </link>
+<xacro:hephaestus prefix="master" reflect="0" />
 <xacro:if value="$(arg twoArm)">
-  <xacro:hephaestus prefix="slave" reflect="-1" />
+  <xacro:hephaestus prefix="slave" reflect="1" />
 </xacro:if>
-<xacro:hephaestus prefix="master" reflect="1" />
 <!-- <xacro:hephaestus prefix="slave" reflect="-1" /> -->
 </robot>
